Commit message: flipped lidar

File: bumperbot_description/urdf/bumperbot.urdf.xacro (robot description, xacro)
@@ -201,5 +201,5 @@
   </link>
   <joint name="laser_joint" type="fixed">
-    <origin xyz="-0.0050526 -0.0023221 0.1208" rpy="0 0 3.14" />
+    <origin xyz="-0.0050526 -0.0023221 0.1208" rpy="0 0 0" />
     <parent link="base_link" />
     <child link="laser_link" />
